Commit message: update urdf for turtle dimensions

File: turtle_description/urdf/khan.urdf.xacro (robot description, xacro)
@@ -27,15 +27,15 @@
   <property name="M_PI" value="3.14159"/>
   <!-- Base Size -->
-  <property name="base_x_size" value="0.245" />
-  <property name="base_y_size" value="0.153" />
-  <property name="base_z_size" value="0.074" />
-  <property name="base_z_clearance" value="0.021" />
+  <property name="base_x_size" value="0.9" />
+  <property name="base_y_size" value="0.42" />
+  <property name="base_z_size" value="0.4" />
+  <property name="base_z_clearance" value="0.17" />
   <!-- Wheel Mounting Positions -->
-  <xacro:property name="wheelbase" value="0.185" />
-  <xacro:property name="track" value="0.189" />
+  <xacro:property name="wheelbase" value="0.762" />
+  <xacro:property name="track" value="0.711" />
   <xacro:property name="wheel_vertical_offset" value="0.0" />
   <!-- Wheel Properties -->
-  <xacro:property name="wheel_length" value="0.036" />
-  <xacro:property name="wheel_radius" value="0.03" />
+  <xacro:property name="wheel_length" value="0.127" />
+  <xacro:property name="wheel_radius" value="0.203" />
   <xacro:macro name="khan_robot">
     <!-- Base link is the center of the robot's base on ground -->
