Commit message: update naming from old robot name to turtle for urdf/description

File: turtle_description/urdf/decorations.urdf.xacro (robot description, xacro)
@@ -21,12 +21,12 @@
 ARISING IN ANY WAY OUT OF THE USE OF THIS SOFTWARE, EVEN IF ADVISED OF THE POSSIBILITY OF SUCH DAMAGE.
 -->
-<robot name="khan_decorations" xmlns:xacro="http://ros.org/wiki/xacro">
-  <xacro:macro name="khan_decorate">
-    <!-- Spawn Khan chassis -->
+<robot name="turtle_decorations" xmlns:xacro="http://ros.org/wiki/xacro">
+  <xacro:macro name="turtle_decorate">
+    <!-- Spawn turtle chassis -->
     <link name="top_chassis_link">
       <visual>
         <origin xyz="0 0 0" rpy="0 0 0" />
         <geometry>
-          <mesh filename="package://khan_description/meshes/top_chassis.stl" />
+          <mesh filename="package://turtle_description/meshes/top_chassis.stl" />
         </geometry>
       </visual>
@@ -41,5 +41,5 @@
       <visual>
         <geometry>
-          <mesh filename="package://khan_description/meshes/user_rail.stl" />
+          <mesh filename="package://turtle_description/meshes/user_rail.stl" />
         </geometry>
       </visual>
@@ -55,5 +55,5 @@
       <visual>
         <geometry>
-          <mesh filename="package://khan_description/meshes/bumper.stl" />
+          <mesh filename="package://turtle_description/meshes/bumper.stl" />
         </geometry>
       </visual>
@@ -69,5 +69,5 @@
       <visual>
         <geometry>
-          <mesh filename="package://khan_description/meshes/bumper.stl" />
+          <mesh filename="package://turtle_description/meshes/bumper.stl" />
         </geometry>
       </visual>
@@ -79,5 +79,5 @@
       <child link="rear_bumper_link" />
     </joint>
-    <xacro:if value="$(optenv KHAN_TOP_PLATE_ENABLED true)">
+    <xacro:if value="$(optenv turtle_TOP_PLATE_ENABLED true)">
       <!-- Spawn the top plate -->
       <link name="top_plate_link">
@@ -85,5 +85,5 @@
           <origin xyz="0 0 0" rpy="0 0 0" />
           <geometry>
-            <mesh filename="package://khan_description/meshes/top_plate.stl" />
+            <mesh filename="package://turtle_description/meshes/top_plate.stl" />
           </geometry>
         </visual>
@@ -91,5 +91,5 @@
           <origin xyz="0 0 0" rpy="0 0 0"/>
           <geometry>
-            <mesh filename="package://khan_description/meshes/top_plate.stl" />
+            <mesh filename="package://turtle_description/meshes/top_plate.stl" />
           </geometry>
         </collision>

File: turtle_description/urdf/description.xacro (robot description, xacro)
@@ -21,6 +21,6 @@
 ARISING IN ANY WAY OUT OF THE USE OF THIS SOFTWARE, EVEN IF ADVISED OF THE POSSIBILITY OF SUCH DAMAGE.
 -->
-<robot name="khan" xmlns:xacro="http://ros.org/wiki/xacro">
-  <xacro:include filename="$(find khan_description)/urdf/khan.urdf.xacro" />
-  <xacro:khan_robot />
+<robot name="leonardo" xmlns:xacro="http://ros.org/wiki/xacro">
+  <xacro:include filename="$(find turtle_description)/urdf/turtle.urdf.xacro" />
+  <xacro:turtle_robot />
 </robot>

File: turtle_description/urdf/turtle.gazebo.xacro (robot description, xacro)
@@ -21,6 +21,6 @@
 ARISING IN ANY WAY OUT OF THE USE OF THIS SOFTWARE, EVEN IF ADVISED OF THE POSSIBILITY OF SUCH DAMAGE.
 -->
-<robot name="khan_robot_gazebo" xmlns:xacro="http://ros.org/wiki/xacro">
-  <xacro:include filename="$(find khan_description)/urdf/khan.urdf.xacro" />
+<robot name="turtle_robot_gazebo" xmlns:xacro="http://ros.org/wiki/xacro">
+  <xacro:include filename="$(find turtle_description)/urdf/turtle.urdf.xacro" />
   <!-- Gazebo plugin for ROS Control -->
   <gazebo>
@@ -29,5 +29,5 @@
     </plugin>
   </gazebo>
-  <xacro:khan_robot />
-  <xacro:khan_robot_gazebo />
+  <xacro:turtle_robot />
+  <xacro:turtle_robot_gazebo />
 </robot>

File: turtle_description/urdf/turtle.urdf.xacro (robot description, xacro)
@@ -2,6 +2,6 @@
 <!--
 Software License Agreement (BSD)
-\file      khan.urdf.xacro
-\authors   Coleman Knabe <csknabe@gmail.com> based on work by Paul Bovbel <pbovbel@clearpathrobotics.com>, Devon Ash <dash@clearpathrobotics.com>
+\file      turtle.urdf.xacro
+\authors  Anthony Wagner based on work by Coleman Knabe <csknabe@gmail.com>, Paul Bovbel <pbovbel@clearpathrobotics.com>, Devon Ash <dash@clearpathrobotics.com>
 \copyright Copyright (c) 2015, Clearpath Robotics, Inc., All rights reserved.
 Redistribution and use in source and binary forms, with or without modification, are permitted provided that
@@ -21,8 +21,8 @@
 ARISING IN ANY WAY OUT OF THE USE OF THIS SOFTWARE, EVEN IF ADVISED OF THE POSSIBILITY OF SUCH DAMAGE.
 -->
-<robot name="khan_robot" xmlns:xacro="http://ros.org/wiki/xacro">
+<robot name="turtle_robot" xmlns:xacro="http://ros.org/wiki/xacro">
   <!-- Included URDF/XACRO Files -->
-  <xacro:include filename="$(find khan_description)/urdf/decorations.urdf.xacro" />
-  <xacro:include filename="$(find khan_description)/urdf/wheel.urdf.xacro" />
+  <xacro:include filename="$(find turtle_description)/urdf/decorations.urdf.xacro" />
+  <xacro:include filename="$(find turtle_description)/urdf/wheel.urdf.xacro" />
   <property name="M_PI" value="3.14159"/>
   <!-- Base Size -->
@@ -38,5 +38,5 @@
   <xacro:property name="wheel_length" value="0.127" />
   <xacro:property name="wheel_radius" value="0.203" />
-  <xacro:macro name="khan_robot">
+  <xacro:macro name="turtle_robot">
     <!-- Base link is the center of the robot's base on ground -->
     <link name="base_link">
@@ -44,5 +44,5 @@
         <origin xyz="0 0 0" rpy="0 0 0" />
         <geometry>
-          <mesh filename="package://khan_description/meshes/rover_base_with_tread.stl" scale="0.001 0.001 0.001"/>
+          <mesh filename="package://turtle_description/meshes/rover_base_with_tread.stl" scale="0.001 0.001 0.001"/>
         </geometry>
       </visual>
@@ -74,18 +74,18 @@
       <child link="inertial_link" />
     </joint>
-    <!-- Khan wheel macros -->
-    <xacro:khan_wheel wheel_prefix="front_left">
+    <!-- turtle wheel macros -->
+    <xacro:turtle_wheel wheel_prefix="front_left">
       <origin xyz="${wheelbase/2} ${track/2} ${wheel_radius}" rpy="0 0 0" />
-    </xacro:khan_wheel>
-    <xacro:khan_wheel wheel_prefix="front_right">
+    </xacro:turtle_wheel>
+    <xacro:turtle_wheel wheel_prefix="front_right">
       <origin xyz="${wheelbase/2} ${-track/2} ${wheel_radius}" rpy="0 0 0" />
-    </xacro:khan_wheel>
-    <xacro:khan_wheel wheel_prefix="rear_left">
+    </xacro:turtle_wheel>
+    <xacro:turtle_wheel wheel_prefix="rear_left">
       <origin xyz="${-wheelbase/2} ${track/2} ${wheel_radius}" rpy="0 0 0" />
-    </xacro:khan_wheel>
-    <xacro:khan_wheel wheel_prefix="rear_right">
+    </xacro:turtle_wheel>
+    <xacro:turtle_wheel wheel_prefix="rear_right">
       <origin xyz="${-wheelbase/2} ${-track/2} ${wheel_radius}" rpy="0 0 0" />
-    </xacro:khan_wheel>
-<!--    <xacro:khan_decorate /> FIXME if we want to put tracks as a decoration rather than part of base-->
+    </xacro:turtle_wheel>
+<!--    <xacro:turtle_decorate /> FIXME if we want to put tracks as a decoration rather than part of base-->
   </xacro:macro>
 </robot>

File: turtle_description/urdf/wheel.urdf.xacro (robot description, xacro)
@@ -21,6 +21,6 @@
 ARISING IN ANY WAY OUT OF THE USE OF THIS SOFTWARE, EVEN IF ADVISED OF THE POSSIBILITY OF SUCH DAMAGE.
 -->
-<robot xmlns:xacro="http://ros.org/wiki/xacro" name="khan_wheel">
-	<xacro:macro name="khan_wheel" params="wheel_prefix *joint_pose">
+<robot xmlns:xacro="http://ros.org/wiki/xacro" name="turtle_wheel">
+	<xacro:macro name="turtle_wheel" params="wheel_prefix *joint_pose">
 		<link name="${wheel_prefix}_wheel_link">
 			<inertial> <!-- FIXME -->
@@ -32,5 +32,5 @@
 				<origin xyz="0 0 0" rpy="0 0 0" />
 				<geometry>
-					<mesh filename="package://khan_description/meshes/rover_wheel.stl" scale="0.001 0.001 0.001" />
+					<mesh filename="package://turtle_description/meshes/rover_wheel.stl" scale="0.001 0.001 0.001" />
 				</geometry>
 			</visual>
